Commit message: docs: Add lidar sensor, remove caster wheel, and refine robot dimensions and joint parameters.

File: examples/diff_drive_robot.urdf (robot description, URDF)
Before this commit: robot diff_drive_robot, 4 links, 3 joints
Links:
- removed link caster_wheel
- added link lidar_link, mass 1; visual cylinder length=0.037866 radius=0.03174
- link base_link: geometry collision box size=0.4 0.3 0.1; visual box size=0.4 0.3 0.1
- link left_wheel: mass 1 -> 0.5
- link right_wheel: mass 1 -> 0.5
Joints:
- removed joint caster_joint
- added joint lidar_link_joint: type fixed, parent base_link, child lidar_link, origin xyz=0 0 0.064282 rpy=0 0 0
- joint left_wheel_joint: limit (none) -> effort=10 velocity=1; origin xyz=0 0.15 0 rpy=-1.570796 0 0 -> xyz=0 0.175 0 rpy=1.570796 0 0
- joint right_wheel_joint: limit (none) -> effort=10 velocity=1; origin xyz=0 -0.15 0 rpy=-1.570796 0 0 -> xyz=0 -0.175 0 rpy=1.570796 0 0
